Commit message: New silia urdf model

File: cob_kuka_description/urdf/kr16/kr16.urdf.xacro (robot description, xacro)
@@ -4,6 +4,6 @@
        xmlns:interface="http://playerstage.sourceforge.net/gazebo/xmlschema/#interface"
        xmlns:xacro="http://ros.org/wiki/xacro">
-	<!--include filename="$(find cob_description)/urdf/lbr/lbr.gazebo.xacro" /-->
-	<!--include filename="$(find cob_description)/urdf/lbr/lbr.transmission.xacro" /-->
+	<include filename="$(find cob_kuka_description)/urdf/kr16/kr16.gazebo.xacro" />
+	<include filename="$(find cob_kuka_description)/urdf/kr16/kr16.transmission.xacro" />
 	<xacro:macro name="cob_kr16" params="parent name *origin">
 		<!-- joint between base_link and arm_0_link -->
@@ -16,5 +16,5 @@
 			<inertial>
 				<origin xyz="0 0 0" rpy="0 0 0"/>
-				<mass value="1.0"/>
+				<mass value="2"/>
 				<inertia ixx="0.01" ixy="0" ixz="0" iyy="0.01" iyz="0" izz="0.01" />
 			</inertial>
@@ -30,5 +30,5 @@
 				<origin xyz="0 0 0" rpy="0 0 0" />
 				<geometry>
-					<box size="0.01 0.01 0.01"/>
+					<mesh filename="package://cob_kuka_description/meshes/kr16/joint_0.stl" />
 				</geometry>
 			</collision>
@@ -49,5 +49,5 @@
 				<origin xyz="0 0 0" rpy="0 0 0" />
 				<!--mass value="5.9907"/-->
-				<mass value="2.0"/>
+				<mass value="2"/>
 				<inertia ixx="0.01" ixy="0" ixz="0" iyy="0.01" iyz="0" izz="0.01" />
 			</inertial>
@@ -56,5 +56,4 @@
 				<geometry>
 					<mesh filename="package://cob_kuka_description/meshes/kr16/joint_1.stl" />
-					<!--cylinder radius="0.060" length="0.30"/-->
 				</geometry>
 				<material name="Orange" />
@@ -63,6 +62,5 @@
 				<origin xyz="0 0 0" rpy="0 0 0" />
 				<geometry>
-					<!--mesh filename="package://cob_kuka_description/meshes/kr16/joint_1_collision.stl" /-->
-					<cylinder radius="0.060" length="0.30"/>
+					<mesh filename="package://cob_kuka_description/meshes/kr16/joint_1.stl" />
 				</geometry>
 			</collision>
@@ -77,11 +75,10 @@
 			<dynamics damping="10" />
 			<limit effort="200" velocity="1.9634" lower="-2.0943" upper="2.0943"/>
-			<safety_controller k_position="20" k_velocity="50" soft_lower_limit="${-2.0943 + 0.01}" 	soft_upper_limit="${2.0943 - 0.01}" />
+			<safety_controller k_position="20" k_velocity="50" soft_lower_limit="${-2.0943 + 0.01}" soft_upper_limit="${2.0943 - 0.01}" />
 		</joint>
 		<link name="${name}_2_link">
 			<inertial>
 				<origin xyz="0 0 0" rpy="0 0 0"/>
-				<!--mass value="5.734939"/-->
-				<mass value="2.0"/>
+				<mass value="2"/>
 				<inertia ixx="0.03" ixy="0" ixz="0" iyy="0.03" iyz="0" izz="0.03" />
 			</inertial>
@@ -90,13 +87,11 @@
 				<geometry>
 					<mesh filename="package://cob_kuka_description/meshes/kr16/joint_2.stl" />
-					<cylinder radius="0.060" length="0.30"/>
-				</geometry>
-				<material name="Black" />
-			</visual>
-			<collision>
-				<origin xyz="0 0 0" rpy="0 0 0" />
-				<geometry>
-					<!--mesh filename="package://cob_kuka_description/meshes/kr16/joint_2_collision.stl"/-->
-					<cylinder radius="0.060" length="0.30"/>
+				</geometry>
+				<material name="Black" />
+			</visual>
+			<collision>
+				<origin xyz="0 0 0" rpy="0 0 0" />
+				<geometry>
+					<mesh filename="package://cob_kuka_description/meshes/kr16/joint_2.stl" />
 				</geometry>
 			</collision>
@@ -116,6 +111,5 @@
 			<inertial>
 				<origin xyz="0 0 0" rpy="0 0 0"/>
-				<!--mass value="4.214668"/-->
-				<mass value="2.0"/>
+				<mass value="2"/>
 				<inertia ixx="0.03" ixy="0" ixz="0" iyy="0.03" iyz="0" izz="0.03" />
 			</inertial>
@@ -124,5 +118,4 @@
 				<geometry>
 					<mesh filename="package://cob_kuka_description/meshes/kr16/joint_3.stl" />
-					<!--cylinder radius="0.060" length="0.30"/-->
 				</geometry>
 				<material name="Orange" />
@@ -131,6 +124,5 @@
 				<origin xyz="0 0 0" rpy="0 0 0" />
 				<geometry>
-					<!--mesh filename="package://cob_kuka_description/meshes/kr16/joint_3_collision.stl"/-->
-					<cylinder radius="0.060" length="0.30"/>
+					<mesh filename="package://cob_kuka_description/meshes/kr16/joint_3.stl" />
 				</geometry>
 			</collision>
@@ -145,5 +137,4 @@
 			<dynamics damping="5" />
 			<limit effort="100" velocity="1.9634" lower="-2.0943" upper="2.0943"/>
-			<!--limit effort="176" velocity="0.4189" upper="2.0943951" lower="-2.0943951"/-->
 			<safety_controller k_position="20" k_velocity="25" soft_lower_limit="${-2.0943 + 0.01}" soft_upper_limit="${2.0943 - 0.01}" />
 		</joint>
@@ -151,6 +142,5 @@
 			<inertial>
 				<origin xyz="0 0 0" rpy="0 0 0"/>
-				<!--mass value="3.669819"/-->
-				<mass value="2.0"/>
+				<mass value="2"/>
 				<inertia ixx="0.03" ixy="0" ixz="0" iyy="0.03" iyz="0" izz="0.03" />
 			</inertial>
@@ -159,13 +149,11 @@
 				<geometry>
 					<mesh filename="package://cob_kuka_description/meshes/kr16/joint_4.stl" />
-					<!--cylinder radius="0.060" length="0.30"/-->
-				</geometry>
-				<material name="Black" />
-			</visual>
-			<collision>
-				<origin xyz="0 0 0" rpy="0 0 0" />
-				<geometry>
-					<!--mesh filename="package://cob_kuka_description/meshes/kr16/joint_4_collision.stl"/-->
-					<cylinder radius="0.060" length="0.30"/>
+				</geometry>
+				<material name="Black" />
+			</visual>
+			<collision>
+				<origin xyz="0 0 0" rpy="0 0 0" />
+				<geometry>
+					<mesh filename="package://cob_kuka_description/meshes/kr16/joint_4.stl" />
 				</geometry>
 			</collision>
@@ -185,5 +173,5 @@
 			<inertial>
 				<origin xyz="0 0 0" rpy="0 0 0"/>
-				<mass value="2.313272"/>
+				<mass value="2"/>
 				<inertia ixx="0.03" ixy="0" ixz="0" iyy="0.03" iyz="0" izz="0.03" />
 			</inertial>
@@ -192,5 +180,4 @@
 				<geometry>
 					<mesh filename="package://cob_kuka_description/meshes/kr16/joint_5.stl" />
-					<!--cylinder radius="0.060" length="0.30"/-->
 				</geometry>
 				<material name="Orange" />
@@ -199,6 +186,5 @@
 				<origin xyz="0 0 0" rpy="0 0 0" />
 				<geometry>
-					<!--mesh filename="package://cob_kuka_description/meshes/kr16/joint_5_collision.stl"/-->
-					<cylinder radius="0.060" length="0.30"/>
+					<mesh filename="package://cob_kuka_description/meshes/kr16/joint_5.stl" />
 				</geometry>
 			</collision>
@@ -206,5 +192,5 @@
 		<!-- joint between arm_5_link and arm_6_link -->
 		<joint name="${name}_6_joint" type="revolute">
-			<origin xyz="0.158 0 -0.1" rpy="0 -${M_PI/2} 0" />  <!--origin xyz="0.115 0 0" rpy="0 -${M_PI/2} 0" /-->
+			<origin xyz="0.158 0 -0.1" rpy="0 -${M_PI/2} 0" />
 			<parent link="${name}_5_link"/>
 			<child link="${name}_6_link"/>
@@ -213,5 +199,4 @@
 			<dynamics damping="5" />
 			<limit effort="30" velocity="1.9634" lower="-2.0943951" upper="2.0943951" />
-			<!--limit effort="20.1" velocity="0.4363" upper="2.0943951" lower="-2.0943951" /-->
 			<safety_controller k_position="20" k_velocity="25" soft_lower_limit="${-2.0943951 + 0.01}" soft_upper_limit="${2.0943951 - 0.01}" />
 		</joint>
@@ -219,5 +204,5 @@
 			<inertial>
 				<origin xyz="0 0 0" rpy="0 0 0"/>
-				<mass value="2.057856"/>
+				<mass value="2"/>
 				<inertia ixx="0.01" ixy="0" ixz="0" iyy="0.01" iyz="0" izz="0.01" />
 			</inertial>
@@ -226,19 +211,17 @@
 				<geometry>
 					<mesh filename="package://cob_kuka_description/meshes/kr16/joint_6.stl" />
-					<!--cylinder radius="0.060" length="0.30"/-->
-				</geometry>
-				<material name="Black" />
-			</visual>
-			<collision>
-				<origin xyz="0 0 0" rpy="0 0 0" />
-				<geometry>
-					<!--mesh filename="package://cob_kuka_description/meshes/kr16/joint_6_collision.stl"/-->
-					<cylinder radius="0.060" length="0.30"/>
+				</geometry>
+				<material name="Black" />
+			</visual>
+			<collision>
+				<origin xyz="0 0 0" rpy="0 0 0" />
+				<geometry>
+					<mesh filename="package://cob_kuka_description/meshes/kr16/joint_6.stl" />
 				</geometry>
 			</collision>
 		</link>
 		<!-- extensions -->
-		<xacro:cob_kr16_gazebo name="${name}" />
-		<xacro:cob_kr16_transmission name="${name}" />
+		<xacro:kr16_gazebo name="${name}" />
+		<xacro:kr16_transmission name="${name}" />
 	</xacro:macro>
 </robot>

File: cob_silia/urdf/silia.urdf (robot description, URDF)
Before this commit: robot silia, 9 links, 8 joints
Links:
- link arm_0_link: geometry collision mesh filename=package://cob_kuka_description/meshes/kr16/joint_0.stl; visual mesh filename=package://cob_kuka_description/meshes/kr16/joint_0.stl
- link arm_1_link: geometry collision mesh filename=package://cob_kuka_description/meshes/kr16/joint_1.stl; visual mesh filename=package://cob_kuka_description/meshes/kr16/joint_1.stl
- link arm_2_link: geometry collision mesh filename=package://cob_kuka_description/meshes/kr16/joint_2.stl; visual mesh filename=package://cob_kuka_description/meshes/kr16/joint_2.stl
- link arm_3_link: geometry collision mesh filename=package://cob_kuka_description/meshes/kr16/joint_3.stl; visual mesh filename=package://cob_kuka_description/meshes/kr16/joint_3.stl
- link arm_4_link: geometry collision mesh filename=package://cob_kuka_description/meshes/kr16/joint_4.stl; visual mesh filename=package://cob_kuka_description/meshes/kr16/joint_4.stl
- link arm_5_link: geometry collision mesh filename=package://cob_kuka_description/meshes/kr16/joint_5.stl; visual mesh filename=package://cob_kuka_description/meshes/kr16/joint_5.stl
- link arm_6_link: geometry collision mesh filename=package://cob_kuka_description/meshes/kr16/joint_6.stl; visual mesh filename=package://cob_kuka_description/meshes/kr16/joint_6.stl
- link stack_link: mass None -> 20; geometry collision mesh filename=package://cob_kuka_description/meshes/kr16/stack.stl; visual mesh filename=package://cob_kuka_description/meshes/kr16/stack.stl
Joints:
- joint arm_0_joint: origin xyz=0 0 0 rpy=0 0 0 -> xyz=0 0 0.6 rpy=0 0 0
- joint stack_joint: origin xyz=1 0.5 0 rpy=0 0 0.785398163397 -> xyz=0 0 0.6 rpy=0 0 3.14159265359

File: cob_silia/urdf/silia.urdf.xacro (robot description, xacro)
@@ -8,8 +8,9 @@
   <include filename="$(find cob_description)/urdf/common.xacro" />
   <include filename="$(find cob_kuka_description)/urdf/materials.urdf.xacro" />
+  <include filename="$(find cob_description)/gazebo/gazebo.urdf.xacro" />
 	<!-- arm mount positions | relative to base_link -->
 	<property name="arm_x" value="0"/>
 	<property name="arm_y" value="0"/>
-	<property name="arm_z" value="0"/>
+	<property name="arm_z" value="0.6"/>
 	<property name="arm_roll" value="0"/>
 	<property name="arm_pitch" value="0"/>
@@ -28,5 +29,5 @@
 		<inertial>
 			<origin xyz="0 0 0" rpy="0 0 0"/>
-			<mass value="1.0"/>
+			<mass value="100.0"/>
 			<inertia ixx="0.01" ixy="0" ixz="0" iyy="0.01" iyz="0" izz="0.01" />
 		</inertial>
@@ -46,9 +47,33 @@
 	<!-- workcell -->
 	<joint name="stack_joint" type="fixed">
-		<origin xyz="1 0.5 0" rpy="0 0 ${M_PI/4}"/>
+		<origin xyz="0 0 0.6" rpy="0 0 ${-3*M_PI/4}"/>
 			<parent link="base_link"/>
 			<child link="stack_link"/>
 		</joint>
-     <link name="stack_link"/>
+		<link name="stack_link">
+			<inertial>
+				<origin xyz="0 0 0" rpy="0 0 0"/>
+				<mass value="100"/>
+				<inertia ixx="0.01" ixy="0" ixz="0" iyy="0.01" iyz="0" izz="0.01" />
+			</inertial>
+			<visual>
+				<origin xyz="0 0 0" rpy="0 0 0" />
+				<geometry>
+					<!--cylinder radius="0.060" length="0.30"/-->
+					<mesh filename="package://cob_kuka_description/meshes/kr16/stack.stl" />
+				</geometry>
+				<material name="Grey" />
+			</visual>
+			<collision>
+				<origin xyz="0 0 0" rpy="0 0 0" />
+				<geometry>
+					<mesh filename="package://cob_kuka_description/meshes/kr16/stack.stl" />
+				</geometry>
+			</collision>
+		</link>
+        <gazebo reference="stack_link">
+                <material>Gazebo/Grey</material>
+                <turnGravityOff>false</turnGravityOff>
+        </gazebo>
   <!-- composition of the robot -->
   <xacro:cob_kr16 name="arm" parent="base_link">
