Commit message: added ik_fast based arm_navigation for silias

File: cob_kuka_description/urdf/kr16/kr16.transmission.xacro (robot description, xacro)
@@ -35,9 +35,4 @@
 			<mechanicalReduction>1</mechanicalReduction>
 		</transmission>
-		<transmission name="${name}_7_trans" type="pr2_mechanism_model/SimpleTransmission">
-			<actuator name="${name}_7_motor"/>
-			<joint name="${name}_7_joint"/>
-			<mechanicalReduction>1</mechanicalReduction>
-		</transmission>
 	</xacro:macro>
 </robot>
