Commit message: Added cfg folder

File: cob_silia/urdf/silia.urdf (robot description, URDF)
Before this commit: robot silia, 9 links, 8 joints
Links:
- added link head_cam3d_link; visual box size=0.1 0.2 0.05
- added link kinect_2_link; visual box size=0.1 0.2 0.05
- link arm_0_link: mass 1.0 -> 2
- link arm_1_link: mass 2.0 -> 2
- link arm_2_link: mass 2.0 -> 2
- link arm_3_link: mass 2.0 -> 2
- link arm_4_link: mass 2.0 -> 2
- link arm_5_link: mass 2.313272 -> 2
- link arm_6_link: mass 2.057856 -> 2
- link base_link: mass 1.0 -> 100.0
- link stack_link: mass 20 -> 100
Joints:
- added joint kinect_1_joint: type fixed, parent base_link, child head_cam3d_link, origin xyz=0 0 0.6 rpy=0 0 0
- added joint kinect_2_joint: type fixed, parent base_link, child kinect_2_link
- joint stack_joint: origin xyz=0 0 0.6 rpy=0 0 3.14159265359 -> xyz=0 0 0.6 rpy=0 0 -3.14159265359

File: cob_silia/urdf/silia.urdf.xacro (robot description, xacro)
@@ -24,4 +24,29 @@
 	<property name="arm_6_ref" value="0.0"/>
 	<property name="arm_7_ref" value="0.0"/>
+  <!-- Cameras -->
+   <link name="head_cam3d_link" >
+       <visual>
+      	<geometry>
+        	<box size="0.1 0.2 0.05"/>
+      	</geometry>
+      	<origin xyz="1.485 0.285 3.05" rpy="1.57 -0.64577 1.57" />
+       </visual>
+   </link>
+   <joint name="kinect_1_joint" type="fixed">
+   	<parent link="base_link" />
+   	<child link="head_cam3d_link" />
+   </joint>
+   <link name="kinect_2_link" >
+       <visual>
+      	<geometry>
+        	<box size="0.1 0.2 0.05"/>
+      	</geometry>
+      	<origin xyz="-0.285 -1.485 3.05" rpy="1.57 0.64577 0" />
+       </visual>
+   </link>
+   <joint name="kinect_2_joint" type="fixed">
+   	<parent link="base_link" />
+   	<child link="kinect_2_link" />
+   </joint>
   <!-- arm -->
   <include filename="$(find cob_kuka_description)/urdf/kr16/kr16.urdf.xacro" />
@@ -47,5 +72,5 @@
 	<!-- workcell -->
 	<joint name="stack_joint" type="fixed">
-		<origin xyz="0 0 0.6" rpy="0 0 ${-3*M_PI/4}"/>
+		<origin xyz="0 0 0.6" rpy="0 0 ${-4*M_PI/4}"/>
 			<parent link="base_link"/>
 			<child link="stack_link"/>
